Commit message: 迭代更新：适配8寸轮毂电机参数，重构阶梯式车身结构以解决物理穿模问题

File: src/manda_description/urdf/fwids_vehicle.urdf (robot description, URDF)
Before this commit: robot four_wheel_independent_drive_and_steering_vehicle, 21 links, 20 joints
Links:
- removed link front_left_wheel_base_link
- removed link front_left_wheel_suspension
- removed link front_right_wheel_base_link
- removed link front_right_wheel_suspension
- removed link rear_left_wheel_base_link
- removed link rear_left_wheel_suspension
- removed link rear_right_wheel_base_link
- removed link rear_right_wheel_suspension
- link body: mass 100.0 -> 30.0; geometry collision box size=0.73 0.28 0.24; visual box size=0.50 0.28 0.12
- link front_left_wheel_rotor: mass 5.0 -> 4.0; geometry collision sphere radius=0.1015; visual cylinder length=0.06 radius=0.1015
- link front_left_wheel_steer: mass 2.0 -> 1.0; geometry visual box size=0.06 0.04 0.10
- link front_right_wheel_rotor: mass 5.0 -> 4.0; geometry collision sphere radius=0.1015; visual cylinder length=0.06 radius=0.1015
- link front_right_wheel_steer: mass 2.0 -> 1.0; geometry visual box size=0.06 0.04 0.10
- link imu_link: geometry visual box size=0.02 0.02 0.01
- link rear_left_wheel_rotor: mass 5.0 -> 4.0; geometry collision sphere radius=0.1015; visual cylinder length=0.06 radius=0.1015
- link rear_left_wheel_steer: mass 2.0 -> 1.0; geometry visual box size=0.06 0.04 0.10
- link rear_right_wheel_rotor: mass 5.0 -> 4.0; geometry collision sphere radius=0.1015; visual cylinder length=0.06 radius=0.1015
- link rear_right_wheel_steer: mass 2.0 -> 1.0; geometry visual box size=0.06 0.04 0.10
Joints:
- removed joint front_left_wheel_joint
- removed joint front_left_wheel_suspension_joint
- removed joint front_right_wheel_joint
- removed joint front_right_wheel_suspension_joint
- removed joint rear_left_wheel_joint
- removed joint rear_left_wheel_suspension_joint
- removed joint rear_right_wheel_joint
- removed joint rear_right_wheel_suspension_joint
- joint base_joint: origin xyz=0 0 0.625 rpy=0 0 0 -> xyz=0 0 0.24 rpy=0 0 0
- joint front_left_wheel_rotor_joint: limit lower=-1e9 upper=1e9 effort=10000 velocity=200 -> effort=10000 velocity=23.5; origin xyz=0 0 -0.225 rpy=-1.57 0 0 -> xyz=0 0 -0.0985 rpy=-1.570796 0 0; type revolute -> continuous
- joint front_left_wheel_steer_joint: origin xyz=0.0 0.0 -0.1 rpy=0 0 0 -> xyz=0.24 0.19 -0.04 rpy=0 0 0; parent front_left_wheel_suspension -> body
- joint front_right_wheel_rotor_joint: limit lower=-1e9 upper=1e9 effort=10000 velocity=200 -> effort=10000 velocity=23.5; origin xyz=0 0 -0.225 rpy=-1.57 0 0 -> xyz=0 0 -0.0985 rpy=-1.570796 0 0; type revolute -> continuous
- joint front_right_wheel_steer_joint: origin xyz=0.0 0.0 -0.1 rpy=0 0 0 -> xyz=0.24 -0.19 -0.04 rpy=0 0 0; parent front_right_wheel_suspension -> body
- joint imu_joint: origin xyz=0 0 0.035 rpy=0 0 0 -> xyz=0 0 0.12 rpy=0 0 0
- joint laser_joint: origin xyz=0.4 0 0.05 rpy=0 0 0 -> xyz=0.3 0 0.13 rpy=0 0 0
- joint rear_left_wheel_rotor_joint: limit lower=-1e9 upper=1e9 effort=10000 velocity=200 -> effort=10000 velocity=23.5; origin xyz=0 0 -0.225 rpy=-1.57 0 0 -> xyz=0 0 -0.0985 rpy=-1.570796 0 0; type revolute -> continuous
- joint rear_left_wheel_steer_joint: origin xyz=0.0 0.0 -0.1 rpy=0 0 0 -> xyz=-0.24 0.19 -0.04 rpy=0 0 0; parent rear_left_wheel_suspension -> body
- joint rear_right_wheel_rotor_joint: limit lower=-1e9 upper=1e9 effort=10000 velocity=200 -> effort=10000 velocity=23.5; origin xyz=0 0 -0.225 rpy=-1.57 0 0 -> xyz=0 0 -0.0985 rpy=-1.570796 0 0; type revolute -> continuous
- joint rear_right_wheel_steer_joint: origin xyz=0.0 0.0 -0.1 rpy=0 0 0 -> xyz=-0.24 -0.19 -0.04 rpy=0 0 0; parent rear_right_wheel_suspension -> body

File: src/manda_description/urdf/fwids_vehicle.xacro (robot description, xacro)
@@ -1,229 +1,226 @@
-<?xml version="1.0"?>
-<robot xmlns:xacro="http://ros.org/wiki/xacro" name="four_wheel_independent_drive_and_steering_vehicle">
-    <xacro:property name="body_mass" value="100.0" />
-    <xacro:property name="body_thickness" value="0.05" />
-    <xacro:property name="tire_mass" value="5.0" />
-    <xacro:property name="tire_radius" value="0.2" />
-    <xacro:property name="tire_thickness" value="0.05" />
-    <xacro:property name="l_f" value="0.5" />
-    <xacro:property name="l_r" value="0.5" />
-    <xacro:property name="d_l" value="0.5" />
-    <xacro:property name="d_r" value="0.5" />
-    <material name="black">  <color rgba="0.2 0.2 0.2 1.0"/> </material>
-    <material name="red">    <color rgba="1.0 0.0 0.0 1.0"/> </material>
-    <material name="blue">   <color rgba="0.0 0.0 1.0 1.0"/> </material>
-    <material name="gray_a"> <color rgba="0.5 0.5 0.5 1.0"/> </material>
-    <xacro:macro name="link_generator" params="name mass color_name *shape *inertia">
-        <link name="${name}">
-            <visual>
-                <geometry><xacro:insert_block name="shape" /></geometry>
-                <material name="${color_name}"/>
-            </visual>
-            <collision>
-                <geometry><xacro:insert_block name="shape" /></geometry>
-            </collision>
-            <inertial>
-                <mass value="${mass}"/>
-                <xacro:insert_block name="inertia" />
-            </inertial>
-        </link>
-    </xacro:macro>
-    <xacro:macro name="fixed_joint" params="name parent child *origin">
-        <joint name="${name}" type="fixed">
-            <xacro:insert_block name="origin" />
-            <parent link="${parent}"/>
-            <child link="${child}"/>
-        </joint>
-    </xacro:macro>
-    <xacro:macro name="wheel_unit" params="name parent x_pos y_pos z_pos">
-        <xacro:link_generator name="${name}_wheel_base_link" mass="1.0" color_name="black">
-            <cylinder radius="0.025" length="0.025" />
-            <inertia ixx="0.005" iyy="0.005" izz="0.005" ixy="0" ixz="0" iyz="0"/>
-        </xacro:link_generator>
-        <xacro:fixed_joint name="${name}_wheel_joint" parent="${parent}" child="${name}_wheel_base_link">
-            <origin xyz="${x_pos} ${y_pos} ${z_pos}" rpy="0 0 0"/>
-        </xacro:fixed_joint>
-        <xacro:link_generator name="${name}_wheel_suspension" mass="1.0" color_name="red">
-            <cylinder radius="0.01" length="0.1"/>
-            <inertia ixx="0.005" iyy="0.005" izz="0.005" ixy="0" ixz="0" iyz="0"/>
-        </xacro:link_generator>
-        <joint name="${name}_wheel_suspension_joint" type="fixed">
-            <origin xyz="0.0 0.0 -0.1" rpy="0 0 0"/>
-            <parent link="${name}_wheel_base_link"/>
-            <child link="${name}_wheel_suspension"/>
-        </joint>
-        <xacro:link_generator name="${name}_wheel_steer" mass="2.0" color_name="gray_a">
-            <cylinder radius="${tire_radius/2.0}" length="${tire_thickness/2.0}"/>
-            <inertia ixx="0.01" iyy="0.01" izz="0.01" ixy="0" ixz="0" iyz="0"/>
-        </xacro:link_generator>
-        <joint name="${name}_wheel_steer_joint" type="revolute">
-            <origin xyz="0.0 0.0 -0.1" rpy="0 0 0"/>
-            <parent link="${name}_wheel_suspension"/>
-            <child link="${name}_wheel_steer"/>
-            <axis xyz="0 0 1"/>
-            <limit effort="1000" velocity="50" lower="-3.1416" upper="3.1416"/>
-            <dynamics damping="10.0" friction="50.0"/>
-        </joint>
-        <xacro:link_generator name="${name}_wheel_rotor" mass="${tire_mass}" color_name="black">
-            <cylinder radius="${tire_radius}" length="${tire_thickness}"/>
-            <inertia ixx="0.051" iyy="0.051" izz="0.1" ixy="0" ixz="0" iyz="0"/>
-        </xacro:link_generator>
-        <joint name="${name}_wheel_rotor_joint" type="revolute">
-            <origin xyz="0 0 ${-tire_radius-0.025}" rpy="-1.57 0 0"/>
-            <parent link="${name}_wheel_steer"/>
-            <child link="${name}_wheel_rotor"/>
-            <axis xyz="0 0 1"/>
-            <limit effort="10000" velocity="200" lower="-1e9" upper="1e9"/>
-            <dynamics damping="50.0" friction="100.0"/>
-        </joint>
-        <gazebo reference="${name}_wheel_rotor">
-            <mu1>5.0</mu1>
-            <mu2>5.0</mu2>
-            <kp>1000000.0</kp>
-            <kd>10.0</kd>
-            <minDepth>0.0001</minDepth>
-            <material>Gazebo/DarkGrey</material>
-        </gazebo>
-    </xacro:macro>
-    <link name="base_footprint"/>
-    <link name="base_link"/>
-    <joint name="footprint_to_base" type="fixed">
-        <origin xyz="0 0 0" rpy="0 0 0"/>
-        <parent link="base_footprint"/>
-        <child link="base_link"/>
-    </joint>
-    <xacro:link_generator name="body" mass="${body_mass}" color_name="gray_a">
-        <cylinder radius="${(l_f + l_r) * 0.5}" length="${body_thickness}" />
-        <inertia ixx="6.2708" iyy="6.2708" izz="12.5" ixy="0" ixz="0" iyz="0"/>
-    </xacro:link_generator>
-    <joint name="base_joint" type="fixed">
-        <origin xyz="0 0 0.625" rpy="0 0 0"/>
-        <parent link="base_link"/>
-        <child link="body"/>
-    </joint>
-    <gazebo reference="body">
-        <material>Gazebo/Grey</material>
+<?xml version="1.0" ?>
+<robot name="four_wheel_independent_drive_and_steering_vehicle" xmlns:xacro="http://www.ros.org/wiki/xacro">
+  <material name="black">
+    <color rgba="0.15 0.15 0.15 1.0"/>
+  </material>
+  <material name="white">
+    <color rgba="0.9 0.9 0.9 1.0"/>
+  </material>
+  <material name="red">
+    <color rgba="1.0 0.0 0.0 1.0"/>
+  </material>
+  <material name="blue">
+    <color rgba="0.0 0.0 1.0 1.0"/>
+  </material>
+  <link name="base_footprint"/>
+  <link name="base_link"/>
+  <joint name="footprint_to_base" type="fixed">
+    <origin rpy="0 0 0" xyz="0 0 0"/>
+    <parent link="base_footprint"/>
+    <child link="base_link"/>
+  </joint>
+  <link name="body">
+    <visual>
+      <origin xyz="0 0 0.06" rpy="0 0 0"/>
+      <geometry><box size="0.73 0.48 0.12"/></geometry>
+      <material name="white"/>
+    </visual>
+    <visual>
+      <origin xyz="0 0 -0.06" rpy="0 0 0"/>
+      <geometry><box size="0.50 0.28 0.12"/></geometry>
+      <material name="black"/>
+    </visual>
+    <collision>
+      <origin xyz="0 0 0" rpy="0 0 0"/>
+      <geometry><box size="0.73 0.28 0.24"/></geometry>
+    </collision>
+    <inertial>
+      <mass value="30.0"/>
+      <inertia ixx="0.72" ixy="0" ixz="0" iyy="1.47" iyz="0" izz="1.90"/>
+    </inertial>
+  </link>
+  <joint name="base_joint" type="fixed">
+    <origin rpy="0 0 0" xyz="0 0 0.24"/>
+    <parent link="base_link"/>
+    <child link="body"/>
+  </joint>
+  <gazebo reference="body">
+    <mu1>0.5</mu1>
+    <mu2>0.5</mu2>
+    <kp>10000000.0</kp>
+    <kd>1.0</kd>
+    <minDepth>0.001</minDepth>
+    <material>Gazebo/White</material>
+  </gazebo>
+  <link name="laser_link">
+    <visual>
+      <geometry><cylinder length="0.025" radius="0.025"/></geometry>
+      <material name="blue"/>
+    </visual>
+    <collision>
+      <geometry><cylinder length="0.025" radius="0.025"/></geometry>
+    </collision>
+    <inertial>
+      <mass value="0.1"/>
+      <inertia ixx="0.0001" ixy="0" ixz="0" iyy="0.0001" iyz="0" izz="0.0001"/>
+    </inertial>
+  </link>
+  <joint name="laser_joint" type="fixed">
+    <origin rpy="0 0 0" xyz="0.3 0 0.13"/> <parent link="body"/>
+    <child link="laser_link"/>
+  </joint>
+  <link name="imu_link">
+    <visual>
+      <geometry><box size="0.02 0.02 0.01"/></geometry>
+      <material name="red"/>
+    </visual>
+    <inertial>
+      <mass value="0.01"/>
+      <inertia ixx="0.00001" ixy="0" ixz="0" iyy="0.00001" iyz="0" izz="0.00001"/>
+    </inertial>
+  </link>
+  <joint name="imu_joint" type="fixed">
+    <origin rpy="0 0 0" xyz="0 0 0.12"/>
+    <parent link="body"/>
+    <child link="imu_link"/>
+  </joint>
+  <xacro:macro name="wheel_module" params="prefix x_offset y_offset">
+    <link name="${prefix}_wheel_steer">
+      <visual>
+        <origin rpy="0 0 0" xyz="0 0 -0.05"/>
+        <geometry><box size="0.06 0.04 0.10"/></geometry>
+        <material name="black"/>
+      </visual>
+      <inertial>
+        <mass value="1.0"/>
+        <inertia ixx="0.005" ixy="0" ixz="0" iyy="0.005" iyz="0" izz="0.005"/>
+      </inertial>
+    </link>
+    <joint name="${prefix}_wheel_steer_joint" type="revolute">
+      <origin rpy="0 0 0" xyz="${x_offset} ${y_offset} -0.04"/>
+      <parent link="body"/>
+      <child link="${prefix}_wheel_steer"/>
+      <axis xyz="0 0 1"/>
+      <limit effort="1000" lower="-3.1416" upper="3.1416" velocity="50"/>
+      <dynamics damping="10.0" friction="50.0"/>
+    </joint>
+    <link name="${prefix}_wheel_rotor">
+      <visual>
+        <geometry>
+          <cylinder length="0.06" radius="0.1015"/>
+        </geometry>
+        <material name="black"/>
+      </visual>
+      <collision>
+        <geometry>
+          <sphere radius="0.1015"/>
+        </geometry>
+      </collision>
+      <inertial>
+        <mass value="4.0"/>
+        <inertia ixx="0.012" ixy="0" ixz="0" iyy="0.012" iyz="0" izz="0.02"/>
+      </inertial>
+    </link>
+    <joint name="${prefix}_wheel_rotor_joint" type="continuous">
+      <origin rpy="-1.570796 0 0" xyz="0 0 -0.0985"/>
+      <parent link="${prefix}_wheel_steer"/>
+      <child link="${prefix}_wheel_rotor"/>
+      <axis xyz="0 0 1"/>
+      <limit effort="10000" velocity="23.5"/>
+      <dynamics damping="1.0" friction="1.0"/>
+    </joint>
+    <gazebo reference="${prefix}_wheel_rotor">
+      <mu1>0.8</mu1>
+      <mu2>0.8</mu2>
+      <kp>10000000.0</kp>
+      <kd>1.0</kd>
+      <minDepth>0.0001</minDepth>
+      <material>Gazebo/DarkGrey</material>
     </gazebo>
-    <xacro:link_generator name="laser_link" mass="0.1" color_name="blue">
-        <cylinder radius="0.025" length="0.025" />
-        <inertia ixx="0.0001" iyy="0.0001" izz="0.0001" ixy="0" ixz="0" iyz="0"/>
-    </xacro:link_generator>
-    <xacro:fixed_joint name="laser_joint" parent="body" child="laser_link">
-        <origin xyz="${(l_f + l_r) * 0.5 * 0.8} 0 ${body_thickness/2.0 + 0.025}" rpy="0 0 0"/>
-    </xacro:fixed_joint>
-    <xacro:link_generator name="imu_link" mass="0.01" color_name="red">
-        <box size="0.02 0.02 0.01" />
-        <inertia ixx="0.00001" iyy="0.00001" izz="0.00001" ixy="0" ixz="0" iyz="0"/>
-    </xacro:link_generator>
-    <xacro:fixed_joint name="imu_joint" parent="body" child="imu_link">
-        <origin xyz="0 0 ${body_thickness/2.0 + 0.005}" rpy="0 0 0"/>
-    </xacro:fixed_joint>
-    <xacro:wheel_unit name="front_left"  parent="body" x_pos="${l_f}"  y_pos="${d_l}"  z_pos="0.0" />
-    <xacro:wheel_unit name="front_right" parent="body" x_pos="${l_f}"  y_pos="${-d_l}" z_pos="0.0" />
-    <xacro:wheel_unit name="rear_left"   parent="body" x_pos="${-l_r}" y_pos="${d_l}"  z_pos="0.0" />
-    <xacro:wheel_unit name="rear_right"  parent="body" x_pos="${-l_r}" y_pos="${-d_l}" z_pos="0.0" />
-    <gazebo reference="laser_link">
-        <material>Gazebo/Blue</material>
-        <sensor type="ray" name="laser">
-            <pose>0 0 0 0 0 0</pose>
-            <visualize>false</visualize>
-            <update_rate>10</update_rate>
-            <ray>
-                <scan>
-                    <horizontal>
-                        <samples>800</samples>
-                        <resolution>1</resolution>
-                        <min_angle>-3.14159</min_angle>
-                        <max_angle>3.14159</max_angle>
-                    </horizontal>
-                </scan>
-                <range>
-                    <min>0.05</min>
-                    <max>30.0</max>
-                    <resolution>0.01</resolution>
-                </range>
-            </ray>
-            <plugin name="gazebo_ros_lidar_controller" filename="libgazebo_ros_ray_sensor.so">
-                <ros><remapping>~/out:=scan</remapping></ros>
-                <output_type>sensor_msgs/LaserScan</output_type>
-                <frame_name>laser_link</frame_name>
-            </plugin>
-        </sensor>
-    </gazebo>
-    <gazebo reference="imu_link">
-        <material>Gazebo/Red</material>
-        <sensor type="imu" name="imu_sensor">
-            <always_on>true</always_on>
-            <update_rate>100</update_rate>
-            <visualize>true</visualize>
-            <plugin filename="libgazebo_ros_imu_sensor.so" name="gazebo_ros_imu_controller">
-                <ros><remapping>~/out:=imu</remapping></ros>
-                <frame_name>imu_link</frame_name>
-            </plugin>
-        </sensor>
-    </gazebo>
-    <gazebo>
-        <plugin name="ground_truth_odometry" filename="libgazebo_ros_p3d.so">
-            <always_on>true</always_on>
-            <update_rate>30.0</update_rate>
-            <ros><remapping>odom:=/groundtruth_odom</remapping></ros>
-            <body_name>base_footprint</body_name>
-            <frame_name>odom</frame_name>
-            <xyz_offset>0 0 0</xyz_offset>
-            <rpy_offset>0 0 0</rpy_offset>
-        </plugin>
-    </gazebo>
-    <xacro:arg name="controller_config_path" default="$(find manda_description)/config/fwids_controllers_ros2.yaml"/>
-    <ros2_control name="GazeboSystem" type="system">
-        <hardware>
-            <plugin>gazebo_ros2_control/GazeboSystem</plugin>
-        </hardware>
-        <joint name="front_left_wheel_steer_joint">
-            <command_interface name="position" />
-            <state_interface name="position" />
-            <state_interface name="velocity" />
-        </joint>
-        <joint name="front_right_wheel_steer_joint">
-            <command_interface name="position" />
-            <state_interface name="position" />
-            <state_interface name="velocity" />
-        </joint>
-        <joint name="rear_left_wheel_steer_joint">
-            <command_interface name="position" />
-            <state_interface name="position" />
-            <state_interface name="velocity" />
-        </joint>
-        <joint name="rear_right_wheel_steer_joint">
-            <command_interface name="position" />
-            <state_interface name="position" />
-            <state_interface name="velocity" />
-        </joint>
-        <joint name="front_left_wheel_rotor_joint">
-            <command_interface name="velocity" />
-            <state_interface name="position" />
-            <state_interface name="velocity" />
-        </joint>
-        <joint name="front_right_wheel_rotor_joint">
-            <command_interface name="velocity" />
-            <state_interface name="position" />
-            <state_interface name="velocity" />
-        </joint>
-        <joint name="rear_left_wheel_rotor_joint">
-            <command_interface name="velocity" />
-            <state_interface name="position" />
-            <state_interface name="velocity" />
-        </joint>
-        <joint name="rear_right_wheel_rotor_joint">
-            <command_interface name="velocity" />
-            <state_interface name="position" />
-            <state_interface name="velocity" />
-        </joint>
-    </ros2_control>
-    <gazebo>
-        <plugin name="gazebo_ros2_control" filename="libgazebo_ros2_control.so">
-            <robot_param>robot_description</robot_param>
-            <robot_param_node>/robot_state_publisher</robot_param_node>
-            <parameters>$(arg controller_config_path)</parameters>
-        </plugin>
-    </gazebo>
+  </xacro:macro>
+  <xacro:wheel_module prefix="front_left" x_offset="0.24" y_offset="0.19" />
+  <xacro:wheel_module prefix="front_right" x_offset="0.24" y_offset="-0.19" />
+  <xacro:wheel_module prefix="rear_left" x_offset="-0.24" y_offset="0.19" />
+  <xacro:wheel_module prefix="rear_right" x_offset="-0.24" y_offset="-0.19" />
+  <gazebo reference="laser_link">
+    <sensor name="laser" type="ray">
+      <pose>0 0 0 0 0 0</pose>
+      <visualize>false</visualize>
+      <update_rate>10</update_rate>
+      <ray>
+        <scan>
+          <horizontal>
+            <samples>800</samples>
+            <resolution>1</resolution>
+            <min_angle>-3.14159</min_angle>
+            <max_angle>3.14159</max_angle>
+          </horizontal>
+        </scan>
+        <range>
+          <min>0.05</min>
+          <max>30.0</max>
+          <resolution>0.01</resolution>
+        </range>
+      </ray>
+      <plugin filename="libgazebo_ros_ray_sensor.so" name="gazebo_ros_lidar_controller">
+        <ros>
+          <remapping>~/out:=scan</remapping>
+        </ros>
+        <output_type>sensor_msgs/LaserScan</output_type>
+        <frame_name>laser_link</frame_name>
+      </plugin>
+    </sensor>
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